File: circuit/数控电源/数控buck.kicad_pcb (KiCad board)
At the start: 2 copper layers, 61.6 x 42.1 mm, 79 parts, among them J1 Conn_01x06_MountingPin, J2 Conn_01x02, J5 Conn_01x02, Q1 BSC070N10NS3G, Q2 BSC070N10NS3G, SW1 SW_Push, U1 STM32F334R8Tx, U2 LM5164DDA, U3 TLV9062, U4 LM5109MA, U5 INA240A1PW, U6 TLV9062, U8 LM2675M-5, Y1 Crystal_GND24

Commit message: 更改原理图，准备改为四开关拓扑
Parts:
- removed C1, C37, C6: 22u, Capacitor_SMD:C_0805_2012Metric_Pad1.18x1.45mm_HandSolder
- removed C10, C26: 10u, Capacitor_SMD:C_0805_2012Metric_Pad1.18x1.45mm_HandSolder
- removed C11, C5: 56p, Capacitor_SMD:C_0603_1608Metric
- removed C12, C13: 470u, Capacitor_SMD:CP_Elec_10x10.5
- removed C14, C16: 12p, Capacitor_SMD:C_0603_1608Metric
- removed C15, C18, C19, C27, C40: 100u, Capacitor_SMD:C_0805_2012Metric_Pad1.18x1.45mm_HandSolder
- removed C2, C7: 10u, Capacitor_SMD:C_1210_3225Metric
- removed C21, C22, C33, C34, C35, C43: 100n, Capacitor_SMD:C_0603_1608Metric
- removed C25: 2.2u, Capacitor_SMD:C_0603_1608Metric
- removed C28, C30: 0.01u, Capacitor_SMD:C_0603_1608Metric_Pad1.08x0.95mm_HandSolder
- removed C3: 2.2n, Capacitor_SMD:C_0603_1608Metric
- removed C31: C_Polarized_US_68u, Capacitor_Tantalum_SMD:CP_EIA-7343-31_Kemet-D
- removed C36: 100nf, Capacitor_SMD:C_0603_1608Metric
- removed C4: 3.3n, Capacitor_SMD:C_0603_1608Metric
- removed C8: 10u, Capacitor_SMD:C_1210_3225Metric_Pad1.33x2.70mm_HandSolder
- removed C9: 1u, Capacitor_SMD:C_0805_2012Metric_Pad1.18x1.45mm_HandSolder
- removed D1, D6: SMCJ58A, Diode_SMD:D_SOD-123F
- removed D13: SS24, Diode_SMD:D_SMA
- removed D2: SS26, Diode_SMD:D_SMA
- removed D3, D4: B5819WS, Diode_SMD:D_SOD-323
- removed D5: LED, LED_SMD:LED_0603_1608Metric_Pad1.05x0.95mm_HandSolder
- removed G***: LOGO, LOGO
- removed J1: Conn_01x06_MountingPin, Connector_JST:JST_GH_SM06B-GHS-TB_1x06-1MP_P1.25mm_Horizontal
- removed J2: Conn_01x02, Connector_AMASS:AMASS_XT30PW-M_1x02_P2.50mm_Horizontal
- removed J5: Conn_01x02, Connector_AMASS:AMASS_XT30PW-F_1x02_P2.50mm_Horizontal
- removed L1: 68u, Inductor_SMD:L_Bourns_SRP7028A_7.3x6.6mm
- removed L2: 33u, Inductor_SMD:L_APV_APH1770
- removed L3: 68u, Inductor_SMD:L_7.3x7.3_H3.5
- removed Q1, Q2: BSC070N10NS3G, Package_TO_SOT_SMD:TDSON-8-1
- removed R1: 100k, Resistor_SMD:R_0603_1608Metric_Pad0.98x0.95mm_HandSolder
- removed R10, R15, R3, R4, R7, R8: 11k, Resistor_SMD:R_0603_1608Metric_Pad0.98x0.95mm_HandSolder
- removed R11: 5m, Resistor_SMD:R_1206_3216Metric_Pad1.30x1.75mm_HandSolder
- removed R12, R13, R14, R5, R6: 1, Resistor_SMD:R_0603_1608Metric_Pad0.98x0.95mm_HandSolder
- removed R16, R19: 27k, Resistor_SMD:R_0603_1608Metric_Pad0.98x0.95mm_HandSolder
- removed R17, R20: 3k, Resistor_SMD:R_0603_1608Metric_Pad0.98x0.95mm_HandSolder
- removed R18: 2, Resistor_SMD:R_0603_1608Metric_Pad0.98x0.95mm_HandSolder
- removed R2: 453k, Resistor_SMD:R_0603_1608Metric_Pad0.98x0.95mm_HandSolder
- removed R9: 11k, Resistor_SMD:R_0603_1608Metric
- removed SW1: SW_Push, Button_Switch_SMD:SW_Push_SPST_NO_Alps_SKRK
- removed U1: STM32F334R8Tx, Package_QFP:LQFP-64_10x10mm_P0.5mm
- removed U2: LM5164DDA, Package_SO:HSOP-8-1EP_3.9x4.9mm_P1.27mm_EP2.41x3.1mm
- removed U3, U6: TLV9062, Package_SO:SOIC-8_3.9x4.9mm_P1.27mm
- removed U4: LM5109MA, Package_SO:SOIC-8_3.9x4.9mm_P1.27mm
- removed U5: INA240A1PW, Package_SO:TSSOP-8_4.4x3mm_P0.65mm
- removed U7: ~, Package_TO_SOT_SMD:SOT-23-5
- removed U8: LM2675M-5, Package_SO:SOIC-8_3.9x4.9mm_P1.27mm
- removed Y1: Crystal_GND24, Crystal:Crystal_SMD_3225-4Pin_3.2x2.5mm_HandSoldering
Routing:
- net +3.3V: track 116.7 -> 0.00 mm, vias 6 -> 0
- net +12V: track 58.9 -> 0.00 mm, vias 1 -> 0
- net /adc_Vin: track 43.2 -> 0.00 mm
- net /HRTIM_-: track 36.2 -> 0.00 mm, vias 2 -> 0
- net /HRTIM_+: track 35.4 -> 0.00 mm, vias 2 -> 0
- net +48V: track 34.8 -> 0.00 mm, vias 1 -> 0
- net GND: track 33.9 -> 0.00 mm, vias 570 -> 0
- net Net-(C4-Pad1): track 28.6 -> 0.00 mm, vias 2 -> 0
- net +5V: track 23.6 -> 0.00 mm
- net /comp_cirurt: track 23.0 -> 0.00 mm, vias 1 -> 0
- net Net-(U2-SW): track 17.6 -> 0.00 mm, vias 2 -> 0
- net Net-(D3-A): track 14.5 -> 0.00 mm, vias 1 -> 0
- net Net-(D4-A): track 14.4 -> 0.00 mm, vias 1 -> 0
- net /comp_volt: track 12.8 -> 0.00 mm
- net +24V: track 12.4 -> 0.00 mm, vias 2 -> 0
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- removed copper zone on F.Cu, net +24V
- removed copper zone on F.Cu, net +48V
- removed copper zone on B.Cu, net GND
- removed copper zone on F.Cu, net GND
- removed copper zone on F.Cu, net Net-(L2-Pad2)
- removed copper zone on B.Cu, net Net-(Q2-D)
- removed copper zone on F.Cu, net Net-(Q2-D)
Other:
- board outline removed
- board text removed: "呆呆"
- board text removed: "数控buck_V2"
