File: circuit/数控电源/数控buck.kicad_sch (KiCad schematic)
At the start: 78 parts, among them J1 Conn_01x06_MountingPin, J2 Conn_01x02, J5 Conn_01x02, Q1 BSC070N10NS3G, Q2 BSC070N10NS3G, SW1 SW_Push, U1 STM32F334R8Tx, U2 LM5164DDA, U3 TLV9062, U4 LM5109MA, U5 INA240A1PW, U6 TLV9062, U8 LM2675M-5, Y1 Crystal_GND24

Commit message: 更改原理图，准备改为四开关拓扑
Parts:
- removed C18: 100u, Capacitor_SMD:C_0805_2012Metric_Pad1.18x1.45mm_HandSolder, symbol Device:C
- removed C31: C_Polarized_US_68u, Capacitor_Tantalum_SMD:CP_EIA-7343-31_Kemet-D, symbol Device:C_Polarized_US
- removed D13: SS24, Diode_SMD:D_SMA, symbol Diode:SS24
- removed L3: 68u, Inductor_SMD:L_7.3x7.3_H3.5, symbol Device:L
- removed U1: STM32F334R8Tx, Package_QFP:LQFP-64_10x10mm_P0.5mm, symbol MCU_ST_STM32F3:STM32F334R8Tx
- removed U8: LM2675M-5, Package_SO:SOIC-8_3.9x4.9mm_P1.27mm, symbol Regulator_Switching:LM2675M-5
- added C17: 10u, Capacitor_SMD:C_0805_2012Metric_Pad1.18x1.45mm_HandSolder, symbol Device:C
- added C18, C31, C39: 470u, Capacitor_SMD:CP_Elec_10x10.5, symbol Device:C_Polarized
- added C20: 100n, Capacitor_SMD:C_0805_2012Metric_Pad1.18x1.45mm_HandSolder, symbol Device:C
- added C23, C24: 100n, Capacitor_SMD:C_0603_1608Metric, symbol Device:C
- added C29, C32: 2.2u, Capacitor_SMD:C_0603_1608Metric, symbol Device:C
- added C38: 1uF, symbol Device:C
- added D7: SS26, Diode_SMD:D_SMA, symbol Diode:SS34
- added D8, D9: B5819WS, Diode_SMD:D_SOD-323, symbol Diode:BAT48JFILM
- added J3: Conn_01x02, symbol Connector_Generic:Conn_01x02
- added L3: 15uH, Library:L_Changjiang_FTC252012S, symbol Library:L
- added Q3, Q4: BSC070N10NS3G, Package_TO_SOT_SMD:TDSON-8-1, symbol Transistor_FET:BSC070N10NS3G
- added R21, R22: 11k, Resistor_SMD:R_0603_1608Metric_Pad0.98x0.95mm_HandSolder, symbol Device:R
- added R23, R24, R25: 1, Resistor_SMD:R_0603_1608Metric_Pad0.98x0.95mm_HandSolder, symbol Device:R
- added R26: 100k, Resistor_SMD:R_01005_0402Metric_Pad0.57x0.30mm_HandSolder, symbol Device:R
- added U1: SIT1057TK-3, Package_DFN_QFN:DFN-8-1EP_3x3mm_P0.65mm_EP1.2x2.15mm, symbol Interface_CAN_LIN:SIT1057TK-3
- added U10: STM32G474RBTx, Package_QFP:LQFP-64_10x10mm_P0.5mm, symbol MCU_ST_STM32G4:STM32G474RBTx
- added U11: PESD1CAN, Package_TO_SOT_SMD:SOT-323_SC-70, symbol Library:PESD1CAN
- added U8: SY8303AIC, library:TSOT-23-8, symbol Library:SY8303AIC
- added U9: LM5109MA, Package_SO:SOIC-8_3.9x4.9mm_P1.27mm, symbol Driver_FET:LM5109MA
- C11: value 56p -> 10n; footprint Capacitor_SMD:C_0603_1608Metric -> Capacitor_SMD:C_0402_1005Metric_Pad0.74x0.62mm_HandSolder
- C14, C16: value 12p -> 18pF; footprint Capacitor_SMD:C_0603_1608Metric -> Capacitor_SMD:C_0402_1005Metric_Pad0.74x0.62mm_HandSolder
- C26: value 10u -> 100nF; footprint Capacitor_SMD:C_0805_2012Metric_Pad1.18x1.45mm_HandSolder -> Capacitor_SMD:C_0402_1005Metric_Pad0.74x0.62mm_HandSolder
- C28: value 0.01u -> 100nF
- C30: value 0.01u -> 10u; footprint Capacitor_SMD:C_0603_1608Metric_Pad1.08x0.95mm_HandSolder -> Capacitor_SMD:C_1210_3225Metric
- C33, C34, C35, C43: footprint Capacitor_SMD:C_0603_1608Metric -> Capacitor_SMD:C_0402_1005Metric_Pad0.74x0.62mm_HandSolder
- C36: value 100nf -> 100nF
- D5: footprint LED_SMD:LED_0603_1608Metric_Pad1.05x0.95mm_HandSolder -> Capacitor_SMD:C_0402_1005Metric_Pad0.74x0.62mm_HandSolder
- R1: footprint Resistor_SMD:R_0603_1608Metric_Pad0.98x0.95mm_HandSolder -> Resistor_SMD:R_01005_0402Metric_Pad0.57x0.30mm_HandSolder
- R10, R15: footprint Resistor_SMD:R_0603_1608Metric_Pad0.98x0.95mm_HandSolder -> Capacitor_SMD:C_0402_1005Metric_Pad0.74x0.62mm_HandSolder
- R19: value 27k -> 220k 0.1%
- R20: value 3k -> 20k 0.1%
- R9: footprint Resistor_SMD:R_0603_1608Metric -> Capacitor_SMD:C_0402_1005Metric_Pad0.74x0.62mm_HandSolder
- U7: value ~ -> (none)
- Y1: frq (none) -> 16Mhz
Connections:
- net +12V: now also C17.1, D7.2 (A), U8.5 (VIN), U9.1 (VDD)
- net +24V: no longer C26.1
- net +3.3V: now also C29.2, U10.1 (VBAT), U10.16 (VDD), U10.29 (VDDA), U10.32 (VDD), U10.48 (VDD), U10.64 (VDD)
- net +48V: now also C30.2, C18.1, C31.1, C39.1, Q3.5 (D)
- net +5V: now also C26.1, C38.1, U1.3 (VCC), U1.5 (VIO)
- net BOOT0: now also U10.7 (PG10)
- net GND: now also C30.1, C17.2, C18.2, C23.1, C24.1, C29.1, C31.2, C32.1, C38.2, C39.2, Q4.1 (S), Q4.2 (S), Q4.3 (S), R21.1, R22.1, R26.2, U1.2 (GND), U1.8 (S), U1.9 (GND), U10.15 (VSS), U10.27 (VSSA), U10.31 (VSS), U10.47 (VSS), U10.63 (VSS), U11.3 (A), U8.3 (GND), U8.4 (GND), U9.4 (VSS); no longer C13.2, C15.2
- net NRST: now also U10.28 (VREF+)
- net OSC_IN: now also U10.5 (PF0)
- net OSC_OUT: now also U10.6 (PF1)
- net SWCLK: now also U10.50 (PA14)
- net SWDIO: now also U10.49 (PA13)
- net adc_Vin: now also C24.2, R25.1, U10.36 (PB14); no longer U3.1, U3.2 (-)
- net adc_volt: now also C32.2, U10.34 (PB12)
- net SW1: now reaches C9.2, L2.1, Q1.1 (S), Q1.2 (S), Q1.3 (S), Q2.5 (D), U4.6 (HS)
- net SW2: now reaches L2.2, R11.1, R12.2
- net SW2: now also C20.2, Q3.1 (S), Q3.2 (S), Q3.3 (S), Q4.5 (D), U9.6 (HS)
- net HRTIM_+ renamed HRTIM1_+
- net HRTIM1_+: now also U10.42 (PA8)
- net HRTIM_- renamed HRTIM1_-
- net HRTIM1_-: now also U10.43 (PA9)
- net USART3_RX renamed UART4_RX
- net UART4_RX: now also U10.53 (PC11)
- net USART3_TX renamed UART4_TX
- net UART4_TX: now also U10.52 (PC10)
- net adc_cir renamed OCP
- net OCP: now also C23.2, U10.33 (PB11), U10.35 (PB13)
- net comp_cirurt: no longer names the net of R14.2, U5.8
- net comp_volt: no longer names the net of R18.1, U6.1, U6.2 (-)
- new net: D8.1 (K), R23.1, U9.7 (HO)
- new net: D8.2 (A), Q3.4 (G), R23.2
- new net: C20.1, D7.1 (K), U9.8 (HB)
- new net: D9.1 (K), R24.1, U9.5 (LO)
- new net: D9.2 (A), Q4.4 (G), R24.2
- new net: R26.1, U8.2 (FS)
- new net: R25.2, U3.1, U3.2 (-)
- new net CAN+: J3.1 (Pin_1), U1.7 (CANH), U11.2 (K)
- new net CAN-: J3.2 (Pin_2), U1.6 (CANL), U11.1 (K)
- new net CAN_RX: U1.1 (TXD), U10.58 (PB5)
- new net CAN_TX: U1.4 (RXD), U10.59 (PB6)
- new net HRTIM2_+: R21.2, U10.44 (PA10), U9.2 (HI)
- new net HRTIM2_-: R22.2, U10.45 (PA11), U9.3 (LI)
- new net I2C_SCL: U10.61 (PB8)
- new net I2C_SDA: U10.60 (PB7)
- new net SPI1_MISO: U10.20 (PA6)
- new net SPI1_MOSI: U10.21 (PA7)
- new net SPI1_SCK: U10.19 (PA5)
- no-connect marks 46 -> 39
Other:
- note added: "12v->5v"
- note removed: "12v to 5v dcdc电路"
- moved on the sheet: C1, C11, C14, C16, C22, C25, C28, C3, C33, C34, C35, C36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

Commit message: 四开关拓扑
Parts:
- added C41: 10nF, Capacitor_SMD:C_0402_1005Metric_Pad0.74x0.62mm_HandSolder, symbol Device:C
- added C42, C44: 22u, Capacitor_SMD:C_0805_2012Metric_Pad1.18x1.45mm_HandSolder, symbol Device:C
- added C45: 10n, Library:C_0402_1005Metric, symbol Library:C
- added R27: 200K±0.1%, Library:R_0402_1005Metric, symbol Library:R
- added R28: 27K±0.1%, Library:R_0402_1005Metric, symbol Library:R
- C25, C29: value 2.2u -> 100nF; footprint Capacitor_SMD:C_0603_1608Metric -> Capacitor_SMD:C_0402_1005Metric_Pad0.74x0.62mm_HandSolder
Connections:
- net +12V: now also U8.8 (EN)
- net +5V: now also L3.2, C42.1, C44.1, C45.1, R27.1
- net GND: now also C13.2, C15.2, C42.2, C44.2, R28.2
- net at L3.1: now also U8.6 (LX), C41.2
- net at U8.1 (FB): now also C45.2, R27.2, R28.1
- net at U8.7 (BS): now also C41.1
Other:
- moved on the sheet: C10, C12, C13, C15, C17, C19, C2, C21, C22, C23, C25, C27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
